Commit message: Flexiv RDK 0.3.1

File: spec/flexiv_rizon4_kinematics.urdf (robot description, URDF)
Before this commit: robot A02L-MP, 9 links, 8 joints
Joints:
- joint joint1: origin xyz=0.0 0.0 0.155 rpy=0 0 3.1415927 -> xyz=0.0 0.0 0.155 rpy=0 0 3.141592653589793
- joint joint4: origin xyz=-0.02 -0.03 0.19 rpy=0 0 -3.1415927 -> xyz=-0.02 -0.03 0.19 rpy=0 0 -3.141592653589793
- joint joint5: origin xyz=-0.02 0.025 0.195 rpy=0 0 -3.1415927 -> xyz=-0.02 0.025 0.195 rpy=0 0 -3.141592653589793
- joint joint7: origin xyz=-0.055 0.070 0.11 rpy=0 -1.5707963 0 -> xyz=-0.055 0.070 0.11 rpy=0 -1.5707963267948966 0
- joint link7_to_flange: origin xyz=0.0 0.0 0.081 rpy=0 0 -3.1415927 -> xyz=0.0 0.0 0.081 rpy=0 0 -3.141592653589793
