Commit message: Update robot description files (#15)
* Update Rizon 4 URDF
* Add Rizon 4s URDF
* Add collision and visual meshes for Rizon 4s
* Replace STL with OBJ for visual meshes

File: resources/flexiv_rizon4s_kinematics.urdf (robot description, URDF)
Before this commit: robot rizon4, 9 links, 8 joints
Links:
- link base_link: geometry collision mesh filename=meshes/rizon4s/collision/link0.stl; visual mesh filename=meshes/rizon4s/visual/link0.obj
- link link1: geometry collision mesh filename=meshes/rizon4s/collision/link1.stl; visual mesh filename=meshes/rizon4s/visual/link1.obj
- link link2: geometry collision mesh filename=meshes/rizon4s/collision/link2.stl; visual mesh filename=meshes/rizon4s/visual/link2.obj
- link link3: geometry collision mesh filename=meshes/rizon4s/collision/link3.stl; visual mesh filename=meshes/rizon4s/visual/link3.obj
- link link4: geometry collision mesh filename=meshes/rizon4s/collision/link4.stl; visual mesh filename=meshes/rizon4s/visual/link4.obj
- link link5: geometry collision mesh filename=meshes/rizon4s/collision/link5.stl; visual mesh filename=meshes/rizon4s/visual/link5.obj
- link link6: geometry collision mesh filename=meshes/rizon4s/collision/link6.stl; visual mesh filename=meshes/rizon4s/visual/link6.obj
- link link7: mass 0.8 -> 1.4; geometry collision mesh filename=meshes/rizon4s/collision/link7.stl; visual mesh filename=meshes/rizon4s/visual/link7.obj
Joints:
- joint link7_to_flange: origin xyz=0.0 0.0 0.081 rpy=0.0 0.0 -3.141592653589793 -> xyz=0.0 0.0 0.124 rpy=0.0 0.0 -3.141592653589793
