Commit message: Update robot name in urdf to "rizon4"

File: resources/flexiv_rizon4_kinematics.urdf (robot description, URDF)
Before this commit: robot A02L-MP, 9 links, 8 joints
Joints:
- joint joint1: origin xyz=0.0 0.0 0.155 rpy=0 0 3.141592653589793 -> xyz=0.0 0.0 0.155 rpy=0.0 0.0 -3.141592653589793
- joint joint2: origin xyz=0.0 0.03 0.210 rpy=0 0 0 -> xyz=0.0 0.03 0.21 rpy=0.0 0.0 0.0
- joint joint3: origin xyz=0.0 0.035 0.205 rpy=0 0 0 -> xyz=0.0 0.035 0.205 rpy=0.0 0.0 0.0
- joint joint4: origin xyz=-0.02 -0.03 0.19 rpy=0 0 -3.141592653589793 -> xyz=-0.02 -0.03 0.19 rpy=0.0 0.0 -3.141592653589793
- joint joint5: origin xyz=-0.02 0.025 0.195 rpy=0 0 -3.141592653589793 -> xyz=-0.02 0.025 0.195 rpy=0.0 0.0 -3.141592653589793
- joint joint6: origin xyz=0.0 0.03 0.19 rpy=0 0 0 -> xyz=0.0 0.03 0.19 rpy=0.0 0.0 0.0
- joint joint7: origin xyz=-0.055 0.070 0.11 rpy=0 -1.5707963267948966 0 -> xyz=-0.055 0.07 0.11 rpy=0.0 -1.5707963478683205 0.0
- joint link7_to_flange: origin xyz=0.0 0.0 0.081 rpy=0 0 -3.141592653589793 -> xyz=0.0 0.0 0.081 rpy=0.0 0.0 -3.141592653589793

Commit message: Replace .stl in visual with .obj

File: resources/flexiv_rizon4_kinematics.urdf (robot description, URDF)
Before this commit: robot rizon4, 9 links, 8 joints
Links:
- link base_link: geometry collision mesh filename=meshes/rizon4/collision/link0.stl; visual mesh filename=meshes/rizon4/visual/link0.obj
- link link1: geometry collision mesh filename=meshes/rizon4/collision/link1.stl; visual mesh filename=meshes/rizon4/visual/link1.obj
- link link2: geometry collision mesh filename=meshes/rizon4/collision/link2.stl; visual mesh filename=meshes/rizon4/visual/link2.obj
- link link3: geometry collision mesh filename=meshes/rizon4/collision/link3.stl; visual mesh filename=meshes/rizon4/visual/link3.obj
- link link4: geometry collision mesh filename=meshes/rizon4/collision/link4.stl; visual mesh filename=meshes/rizon4/visual/link4.obj
- link link5: geometry collision mesh filename=meshes/rizon4/collision/link5.stl; visual mesh filename=meshes/rizon4/visual/link5.obj
- link link6: geometry collision mesh filename=meshes/rizon4/collision/link6.stl; visual mesh filename=meshes/rizon4/visual/link6.obj
- link link7: geometry collision mesh filename=meshes/rizon4/collision/link7.stl; visual mesh filename=meshes/rizon4/visual/link7.obj

Commit message: Update Rizon4 urdf and meshes

File: resources/flexiv_rizon4_kinematics.urdf (robot description, URDF)
Before this commit: robot rizon4, 9 links, 8 joints
Links:
- link flange: mass None -> 0.0
- link link1: geometry collision mesh filename=meshes/rizon4/collision/link1.stl; visual mesh filename=meshes/rizon4/visual/link1.obj
- link link2: geometry collision mesh filename=meshes/rizon4/collision/link2.stl; visual mesh filename=meshes/rizon4/visual/link2.obj
- link link3: geometry collision mesh filename=meshes/rizon4/collision/link3.stl; visual mesh filename=meshes/rizon4/visual/link3.obj
- link link4: geometry collision mesh filename=meshes/rizon4/collision/link4.stl; visual mesh filename=meshes/rizon4/visual/link4.obj
- link link5: geometry collision mesh filename=meshes/rizon4/collision/link5.stl; visual mesh filename=meshes/rizon4/visual/link5.obj
- link link6: mass 2.1 -> 2.2; geometry collision mesh filename=meshes/rizon4/collision/link6.stl; visual mesh filename=meshes/rizon4/visual/link6.obj
- link link7: geometry collision mesh filename=meshes/rizon4/collision/link7.stl; visual mesh filename=meshes/rizon4/visual/link7.obj
Joints:
- joint joint7: origin xyz=-0.055 0.07 0.11 rpy=0.0 -1.5707963478683205 0.0 -> xyz=-0.015 0.073 0.11 rpy=0.0 -1.5707963478683205 0.0

Commit message: Update rizon4s urdf and meshes

File: resources/flexiv_rizon4_kinematics.urdf (robot description, URDF)
Before this commit: robot rizon4, 9 links, 8 joints
Links:
- link base_link: geometry collision mesh filename=package://meshes/collision/link0.stl; visual mesh filename=package://meshes/visual/link0.obj
- link flange: mass 0.0 -> None
- link link1: geometry collision mesh filename=package://meshes/collision/link1.stl; visual mesh filename=package://meshes/visual/link1.obj
- link link2: geometry collision mesh filename=package://meshes/collision/link2.stl; visual mesh filename=package://meshes/visual/link2.obj
- link link3: geometry collision mesh filename=package://meshes/collision/link3.stl; visual mesh filename=package://meshes/visual/link3.obj
- link link4: geometry collision mesh filename=package://meshes/collision/link4.stl; visual mesh filename=package://meshes/visual/link4.obj
- link link5: geometry collision mesh filename=package://meshes/collision/link5.stl; visual mesh filename=package://meshes/visual/link5.obj
- link link6: geometry collision mesh filename=package://meshes/collision/link6.stl; visual mesh filename=package://meshes/visual/link6.obj
- link link7: geometry collision mesh filename=package://meshes/collision/link7.stl; visual mesh filename=package://meshes/visual/link7.obj

File: resources/flexiv_rizon4s_kinematics.urdf (robot description, URDF)
Before this commit: robot rizon4s, 9 links, 8 joints
Links:
- link base_link: geometry collision mesh filename=package://meshes/collision/link0.stl; visual mesh filename=package://meshes/visual/link0.obj
- link link1: geometry collision mesh filename=package://meshes/collision/link1.stl; visual mesh filename=package://meshes/visual/link1.obj
- link link2: geometry collision mesh filename=package://meshes/collision/link2.stl; visual mesh filename=package://meshes/visual/link2.obj
- link link3: geometry collision mesh filename=package://meshes/collision/link3.stl; visual mesh filename=package://meshes/visual/link3.obj
- link link4: geometry collision mesh filename=package://meshes/collision/link4.stl; visual mesh filename=package://meshes/visual/link4.obj
- link link5: geometry collision mesh filename=package://meshes/collision/link5.stl; visual mesh filename=package://meshes/visual/link5.obj
- link link6: mass 2.1 -> 2.2; geometry collision mesh filename=package://meshes/collision/link6.stl; visual mesh filename=package://meshes/visual/link6.obj
- link link7: geometry collision mesh filename=package://meshes/collision/link7.stl; visual mesh filename=package://meshes/visual/link7.obj
Joints:
- joint joint7: origin xyz=-0.055 0.07 0.11 rpy=0.0 -1.5707963478683205 0.0 -> xyz=-0.015 0.073 0.11 rpy=0.0 -1.5707963478683205 0.0
