Commit message: Add Rizon 10 URDF

File: resources/flexiv_rizon10_kinematics.urdf (robot description, URDF)
Before this commit: robot rizon4s, 9 links, 8 joints
Links:
- link base_link: mass 3.7 -> 9.2; geometry collision mesh filename=meshes/rizon10/collision/link0.stl; visual mesh filename=meshes/rizon10/visual/link0.obj
- link link1: mass 3.7 -> 9.7; geometry collision mesh filename=meshes/rizon10/collision/link1.stl; visual mesh filename=meshes/rizon10/visual/link1.obj
- link link2: mass 2.7 -> 6.2; geometry collision mesh filename=meshes/rizon10/collision/link2.stl; visual mesh filename=meshes/rizon10/visual/link2.obj
- link link3: mass 2.4 -> 4.6; geometry collision mesh filename=meshes/rizon10/collision/link3.stl; visual mesh filename=meshes/rizon10/visual/link3.obj
- link link4: mass 2.4 -> 3.0; geometry collision mesh filename=meshes/rizon10/collision/link4.stl; visual mesh filename=meshes/rizon10/visual/link4.obj
- link link5: geometry collision mesh filename=meshes/rizon10/collision/link5.stl; visual mesh filename=meshes/rizon10/visual/link5.obj
- link link6: mass 2.1 -> 2.3; geometry collision mesh filename=meshes/rizon10/collision/link6.stl; visual mesh filename=meshes/rizon10/visual/link6.obj
- link link7: mass 1.4 -> 0.9; geometry collision mesh filename=meshes/rizon10/collision/link7.stl; visual mesh filename=meshes/rizon10/visual/link7.obj
Joints:
- joint joint1: limit lower=-2.7925 upper=2.7925 effort=123 velocity=2.0944 -> lower=-2.7925 upper=2.7925 effort=261 velocity=1.7453; origin xyz=0.0 0.0 0.155 rpy=0.0 0.0 -3.141592653589793 -> xyz=0.0 0.0 0.21 rpy=0.0 0.0 -3.141592653589793
- joint joint2: limit lower=-2.2689 upper=2.2689 effort=123 velocity=2.0944 -> lower=-2.6704 upper=2.6704 effort=261 velocity=1.7453; origin xyz=0.0 0.03 0.21 rpy=0.0 0.0 0.0 -> xyz=0.0 0.0675 0.24 rpy=0.0 0.0 0.0
- joint joint3: limit lower=-2.9671 upper=2.9671 effort=64 velocity=2.4435 -> lower=-2.7925 upper=2.7925 effort=123 velocity=2.0944; origin xyz=0.0 0.035 0.205 rpy=0.0 0.0 0.0 -> xyz=0.0 0.0625 0.2275 rpy=0.0 0.0 0.0
- joint joint4: limit lower=-1.8675 upper=2.6878 effort=64 velocity=2.4435 -> lower=-2.7053 upper=2.7053 effort=123 velocity=2.0944; origin xyz=-0.02 -0.03 0.19 rpy=0.0 0.0 -3.141592653589793 -> xyz=0.0 -0.0625 0.2225 rpy=0.0 0.0 -3.141592653589793
- joint joint5: limit lower=-2.9671 upper=2.9671 effort=39 velocity=4.8869 -> lower=-2.9671 upper=2.9671 effort=57 velocity=3.8397; origin xyz=-0.02 0.025 0.195 rpy=0.0 0.0 -3.141592653589793 -> xyz=0.0 0.0575 0.205 rpy=0.0 0.0 -3.141592653589793
- joint joint6: limit lower=-1.3963 upper=4.5379 effort=39 velocity=4.8869 -> lower=-1.3963 upper=4.5379 effort=57 velocity=3.8397
- joint joint7: limit lower=-2.9671 upper=2.9671 effort=39 velocity=4.8869 -> lower=-2.9671 upper=2.9671 effort=57 velocity=3.8397; origin xyz=-0.055 0.07 0.11 rpy=0.0 -1.5707963478683205 0.0 -> xyz=-0.015 0.073 0.11 rpy=0.0 -1.5707963478683205 0.0
- joint link7_to_flange: origin xyz=0.0 0.0 0.124 rpy=0.0 0.0 -3.141592653589793 -> xyz=0.0 0.0 0.081 rpy=0.0 0.0 -3.141592653589793

Commit message: Update rizon10 urdf and mesh

File: resources/flexiv_rizon10_kinematics.urdf (robot description, URDF)
Before this commit: robot rizon10, 9 links, 8 joints
Links:
- link base_link: geometry collision mesh filename=package://meshes/collision/link0.stl; visual mesh filename=package://meshes/visual/link0.obj
- link link1: geometry collision mesh filename=package://meshes/collision/link1.stl; visual mesh filename=package://meshes/visual/link1.obj
- link link2: geometry collision mesh filename=package://meshes/collision/link2.stl; visual mesh filename=package://meshes/visual/link2.obj
- link link3: geometry collision mesh filename=package://meshes/collision/link3.stl; visual mesh filename=package://meshes/visual/link3.obj
- link link4: geometry collision mesh filename=package://meshes/collision/link4.stl; visual mesh filename=package://meshes/visual/link4.obj
- link link5: geometry collision mesh filename=package://meshes/collision/link5.stl; visual mesh filename=package://meshes/visual/link5.obj
- link link6: geometry collision mesh filename=package://meshes/collision/link6.stl; visual mesh filename=package://meshes/visual/link6.obj
- link link7: geometry collision mesh filename=package://meshes/collision/link7.stl; visual mesh filename=package://meshes/visual/link7.obj

Commit message: Up

File: resources/flexiv_rizon10_kinematics.urdf (robot description, URDF)
Before this commit: robot rizon10, 9 links, 8 joints
Links:
- link base_link: geometry collision mesh filename=package://meshes/rizon10/collision/link0.stl; visual mesh filename=package://meshes/rizon10/visual/link0.obj
- link link1: geometry collision mesh filename=package://meshes/rizon10/collision/link1.stl; visual mesh filename=package://meshes/rizon10/visual/link1.obj
- link link2: geometry collision mesh filename=package://meshes/rizon10/collision/link2.stl; visual mesh filename=package://meshes/rizon10/visual/link2.obj
- link link3: geometry collision mesh filename=package://meshes/rizon10/collision/link3.stl; visual mesh filename=package://meshes/rizon10/visual/link3.obj
- link link4: geometry collision mesh filename=package://meshes/rizon10/collision/link4.stl; visual mesh filename=package://meshes/rizon10/visual/link4.obj
- link link5: geometry collision mesh filename=package://meshes/rizon10/collision/link5.stl; visual mesh filename=package://meshes/rizon10/visual/link5.obj
- link link6: geometry collision mesh filename=package://meshes/rizon10/collision/link6.stl; visual mesh filename=package://meshes/rizon10/visual/link6.obj
- link link7: geometry collision mesh filename=package://meshes/rizon10/collision/link7.stl; visual mesh filename=package://meshes/rizon10/visual/link7.obj

File: resources/flexiv_rizon10s_kinematics.urdf (robot description, URDF)
Before this commit: robot rizon10s, 9 links, 8 joints
Links:
- link base_link: geometry collision mesh filename=package://meshes/rizon10s/collision/link0.stl; visual mesh filename=package://meshes/rizon10s/visual/link0.obj
- link link1: geometry collision mesh filename=package://meshes/rizon10s/collision/link1.stl; visual mesh filename=package://meshes/rizon10s/visual/link1.obj
- link link2: geometry collision mesh filename=package://meshes/rizon10s/collision/link2.stl; visual mesh filename=package://meshes/rizon10s/visual/link2.obj
- link link3: geometry collision mesh filename=package://meshes/rizon10s/collision/link3.stl; visual mesh filename=package://meshes/rizon10s/visual/link3.obj
- link link4: geometry collision mesh filename=package://meshes/rizon10s/collision/link4.stl; visual mesh filename=package://meshes/rizon10s/visual/link4.obj
- link link5: geometry collision mesh filename=package://meshes/rizon10s/collision/link5.stl; visual mesh filename=package://meshes/rizon10s/visual/link5.obj
- link link6: geometry collision mesh filename=package://meshes/rizon10s/collision/link6.stl; visual mesh filename=package://meshes/rizon10s/visual/link6.obj
- link link7: geometry collision mesh filename=package://meshes/rizon10s/collision/link7.stl; visual mesh filename=package://meshes/rizon10s/visual/link7.obj

File: resources/flexiv_rizon4_kinematics.urdf (robot description, URDF)
Before this commit: robot rizon4, 9 links, 8 joints
Links:
- link base_link: geometry collision mesh filename=package://meshes/rizon4/collision/link0.stl; visual mesh filename=package://meshes/rizon4/visual/link0.obj
- link link1: geometry collision mesh filename=package://meshes/rizon4/collision/link1.stl; visual mesh filename=package://meshes/rizon4/visual/link1.obj
- link link2: geometry collision mesh filename=package://meshes/rizon4/collision/link2.stl; visual mesh filename=package://meshes/rizon4/visual/link2.obj
- link link3: geometry collision mesh filename=package://meshes/rizon4/collision/link3.stl; visual mesh filename=package://meshes/rizon4/visual/link3.obj
- link link4: geometry collision mesh filename=package://meshes/rizon4/collision/link4.stl; visual mesh filename=package://meshes/rizon4/visual/link4.obj
- link link5: geometry collision mesh filename=package://meshes/rizon4/collision/link5.stl; visual mesh filename=package://meshes/rizon4/visual/link5.obj
- link link6: geometry collision mesh filename=package://meshes/rizon4/collision/link6.stl; visual mesh filename=package://meshes/rizon4/visual/link6.obj
- link link7: geometry collision mesh filename=package://meshes/rizon4/collision/link7.stl; visual mesh filename=package://meshes/rizon4/visual/link7.obj

File: resources/flexiv_rizon4s_kinematics.urdf (robot description, URDF)
Before this commit: robot rizon4s, 9 links, 8 joints
Links:
- link base_link: geometry collision mesh filename=package://meshes/rizon4s/collision/link0.stl; visual mesh filename=package://meshes/rizon4s/visual/link0.obj
- link link1: geometry collision mesh filename=package://meshes/rizon4s/collision/link1.stl; visual mesh filename=package://meshes/rizon4s/visual/link1.obj
- link link2: geometry collision mesh filename=package://meshes/rizon4s/collision/link2.stl; visual mesh filename=package://meshes/rizon4s/visual/link2.obj
- link link3: geometry collision mesh filename=package://meshes/rizon4s/collision/link3.stl; visual mesh filename=package://meshes/rizon4s/visual/link3.obj
- link link4: geometry collision mesh filename=package://meshes/rizon4s/collision/link4.stl; visual mesh filename=package://meshes/rizon4s/visual/link4.obj
- link link5: geometry collision mesh filename=package://meshes/rizon4s/collision/link5.stl; visual mesh filename=package://meshes/rizon4s/visual/link5.obj
- link link6: geometry collision mesh filename=package://meshes/rizon4s/collision/link6.stl; visual mesh filename=package://meshes/rizon4s/visual/link6.obj
- link link7: geometry collision mesh filename=package://meshes/rizon4s/collision/link7.stl; visual mesh filename=package://meshes/rizon4s/visual/link7.obj
