Commit message: Feature/update robot description (#49)
* Update Rizon4 urdf and meshes
* Update rizon4s urdf and meshes
* Update rizon10 urdf and meshes
* Add rizon10s urdf and meshes

File: resources/flexiv_rizon10s_kinematics.urdf (robot description, URDF)
Before this commit: robot rizon10, 9 links, 8 joints
Links:
- link base_link: geometry collision mesh filename=package://meshes/rizon10s/collision/link0.stl; visual mesh filename=package://meshes/rizon10s/visual/link0.obj
- link link1: geometry collision mesh filename=package://meshes/rizon10s/collision/link1.stl; visual mesh filename=package://meshes/rizon10s/visual/link1.obj
- link link2: geometry collision mesh filename=package://meshes/rizon10s/collision/link2.stl; visual mesh filename=package://meshes/rizon10s/visual/link2.obj
- link link3: geometry collision mesh filename=package://meshes/rizon10s/collision/link3.stl; visual mesh filename=package://meshes/rizon10s/visual/link3.obj
- link link4: geometry collision mesh filename=package://meshes/rizon10s/collision/link4.stl; visual mesh filename=package://meshes/rizon10s/visual/link4.obj
- link link5: geometry collision mesh filename=package://meshes/rizon10s/collision/link5.stl; visual mesh filename=package://meshes/rizon10s/visual/link5.obj
- link link6: geometry collision mesh filename=package://meshes/rizon10s/collision/link6.stl; visual mesh filename=package://meshes/rizon10s/visual/link6.obj
- link link7: mass 0.9 -> 1.5; geometry collision mesh filename=package://meshes/rizon10s/collision/link7.stl; visual mesh filename=package://meshes/rizon10s/visual/link7.obj
Joints:
- joint link7_to_flange: origin xyz=0.0 0.0 0.081 rpy=0.0 0.0 -3.141592653589793 -> xyz=0.0 0.0 0.124 rpy=0.0 0.0 -3.141592653589793

File: resources/flexiv_rizon4_kinematics.urdf (robot description, URDF)
Before this commit: robot rizon4, 9 links, 8 joints
Links:
- link base_link: geometry collision mesh filename=package://meshes/rizon4/collision/link0.stl; visual mesh filename=package://meshes/rizon4/visual/link0.obj
- link link1: geometry collision mesh filename=package://meshes/rizon4/collision/link1.stl; visual mesh filename=package://meshes/rizon4/visual/link1.obj
- link link2: geometry collision mesh filename=package://meshes/rizon4/collision/link2.stl; visual mesh filename=package://meshes/rizon4/visual/link2.obj
- link link3: geometry collision mesh filename=package://meshes/rizon4/collision/link3.stl; visual mesh filename=package://meshes/rizon4/visual/link3.obj
- link link4: geometry collision mesh filename=package://meshes/rizon4/collision/link4.stl; visual mesh filename=package://meshes/rizon4/visual/link4.obj
- link link5: geometry collision mesh filename=package://meshes/rizon4/collision/link5.stl; visual mesh filename=package://meshes/rizon4/visual/link5.obj
- link link6: mass 2.1 -> 2.2; geometry collision mesh filename=package://meshes/rizon4/collision/link6.stl; visual mesh filename=package://meshes/rizon4/visual/link6.obj
- link link7: geometry collision mesh filename=package://meshes/rizon4/collision/link7.stl; visual mesh filename=package://meshes/rizon4/visual/link7.obj
Joints:
- joint joint7: origin xyz=-0.055 0.07 0.11 rpy=0.0 -1.5707963478683205 0.0 -> xyz=-0.015 0.073 0.11 rpy=0.0 -1.5707963478683205 0.0

File: resources/flexiv_rizon4s_kinematics.urdf (robot description, URDF)
Before this commit: robot rizon4s, 9 links, 8 joints
Links:
- link base_link: geometry collision mesh filename=package://meshes/rizon4s/collision/link0.stl; visual mesh filename=package://meshes/rizon4s/visual/link0.obj
- link link1: geometry collision mesh filename=package://meshes/rizon4s/collision/link1.stl; visual mesh filename=package://meshes/rizon4s/visual/link1.obj
- link link2: geometry collision mesh filename=package://meshes/rizon4s/collision/link2.stl; visual mesh filename=package://meshes/rizon4s/visual/link2.obj
- link link3: geometry collision mesh filename=package://meshes/rizon4s/collision/link3.stl; visual mesh filename=package://meshes/rizon4s/visual/link3.obj
- link link4: geometry collision mesh filename=package://meshes/rizon4s/collision/link4.stl; visual mesh filename=package://meshes/rizon4s/visual/link4.obj
- link link5: geometry collision mesh filename=package://meshes/rizon4s/collision/link5.stl; visual mesh filename=package://meshes/rizon4s/visual/link5.obj
- link link6: mass 2.1 -> 2.2; geometry collision mesh filename=package://meshes/rizon4s/collision/link6.stl; visual mesh filename=package://meshes/rizon4s/visual/link6.obj
- link link7: geometry collision mesh filename=package://meshes/rizon4s/collision/link7.stl; visual mesh filename=package://meshes/rizon4s/visual/link7.obj
Joints:
- joint joint7: origin xyz=-0.055 0.07 0.11 rpy=0.0 -1.5707963478683205 0.0 -> xyz=-0.015 0.073 0.11 rpy=0.0 -1.5707963478683205 0.0
